File: kicad/un1eet_sao.kicad_pcb (KiCad board)
At the start: 2 copper layers, 98.1 x 27.3 mm, 4 parts

Commit message: adding sao connector
Parts:
- added J2: #badgelife, un1eet_sao:Badgelife-Shitty-2x2, F.Cu at (132.7, 85.3)
- moved ? 186.8 mm to (153.1, 107.2) (x4)
Other:
- board size 98.1 x 27.3 mm -> 98.1 x 32.3 mm

Commit message: Added a shitty led
Parts:
- added D1: LED, LEDs:LED_0603_HandSoldering, F.Cu at (118.7, 90.2)
- added R1: 330R, Resistors_SMD:R_0603_HandSoldering, F.Cu at (113.0, 86.4)
- turned ? to 90 degrees
Connections:
- J2 pad 1: (no net) -> Net-(J1-Pad1)
- J2 pad 2: (no net) -> GND
Routing:
- net Net-(J1-Pad1): track 0.00 -> 27.1 mm
- net GND: track 0.00 -> 16.6 mm
- net Net-(D1-Pad2): track 0.00 -> 7.94 mm
Changed lines of the file:
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@@
 (kicad_pcb (version 4) (host pcbnew 4.0.7)
   (general
-    (links 0)
+    (links 3)
     (no_connects 0)
     (area 103.86345 78.232405 202.022987 110.591786)
     (thickness 1.6)
     (drawings 1057)
-    (tracks 0)
+    (tracks 25)
     (zones 0)
-    (modules 5)
-    (nets 1)
+    (modules 7)
+    (nets 4)
   )
   (page A4)
@@
     (mod_text_size 1 1)
     (mod_text_width 0.15)
-    (pad_size 1.524 1.524)
-    (pad_drill 0.762)
+    (pad_size 1.7 1.7)
+    (pad_drill 1)
     (pad_to_mask_clearance 0.2)
     (aux_axis_origin 0 0)
@@
   )
   (net 0 "")
+  (net 1 GND)
+  (net 2 "Net-(D1-Pad2)")
+  (net 3 "Net-(J1-Pad1)")
   (net_class Default "This is the default net class."
     (clearance 0.2)
@@
     (uvia_dia 0.3)
     (uvia_drill 0.1)
+    (add_net GND)
+    (add_net "Net-(D1-Pad2)")
+    (add_net "Net-(J1-Pad1)")
   )
   (module un1eet_sao:B.Silk_g8163 (layer F.Cu)
@@
     (pad 4 thru_hole circle (at 1.27 -1.27) (size 1.7 1.7) (drill 1) (layers *.Cu *.Mask))
     (pad 3 thru_hole oval (at 1.27 1.27) (size 1.7 1.7) (drill 1) (layers *.Cu *.Mask))
-    (pad 1 thru_hole oval (at -1.27 -1.27) (size 1.7 1.7) (drill 1) (layers *.Cu *.Mask))
-    (pad 2 thru_hole oval (at -1.27 1.27) (size 1.7 1.7) (drill 1) (layers *.Cu *.Mask))
+    (pad 1 thru_hole oval (at -1.27 -1.27) (size 1.7 1.7) (drill 1) (layers *.Cu *.Mask)
+      (net 3 "Net-(J1-Pad1)"))
+    (pad 2 thru_hole oval (at -1.27 1.27) (size 1.7 1.7) (drill 1) (layers *.Cu *.Mask)
+      (net 1 GND))
   )
   (module un1eet_sao:F.Cu_g8165 (layer F.Cu)
-    (at 153.05 107.17)
-    (fp_text reference "" (at 0 0) (layer F.SilkS)
+    (at 153.05 107.17 90)
+    (fp_text reference "" (at 0 0 90) (layer F.SilkS)
       (effects (font (thickness 0.15)))
     )
-    (fp_text value "" (at 0 0) (layer F.SilkS)
+    (fp_text value "" (at 0 0 90) (layer F.SilkS)
       (effects (font (thickness 0.15)))
     )
@@
       (xy 25.929167 -10.392833) (xy 27.2415 -10.392833) (xy 27.633092 -10.392878) (xy 27.951351 -10.391083)) (layer F.SilkS) (width 0.01))
   )
+  (module Resistors_SMD:R_0603_HandSoldering (layer F.Cu)
+    (at 113.03 86.36 180)
+    (descr "Resistor SMD 0603, hand soldering")
+    (tags "resistor 0603")
+    (attr smd)
+    (fp_text reference R1 (at 0 -1.45 180) (layer F.SilkS)
+      (effects (font (size 1 1) (thickness 0.15)))
+    )
+    (fp_text value 330R (at 0 1.55 180) (layer F.Fab)
+      (effects (font (size 1 1) (thickness 0.15)))
+    )
+    (fp_text user %R (at 0 0 180) (layer F.Fab)
+      (effects (font (size 0.4 0.4) (thickness 0.075)))
+    )
+    (fp_line (start -0.8 0.4) (end -0.8 -0.4) (layer F.Fab) (width 0.1))
+    (fp_line (start 0.8 0.4) (end -0.8 0.4) (layer F.Fab) (width 0.1))
+    (fp_line (start 0.8 -0.4) (end 0.8 0.4) (layer F.Fab) (width 0.1))
+    (fp_line (start -0.8 -0.4) (end 0.8 -0.4) (layer F.Fab) (width 0.1))
+    (fp_line (start 0.5 0.68) (end -0.5 0.68) (layer F.SilkS) (width 0.12))
+    (fp_line (start -0.5 -0.68) (end 0.5 -0.68) (layer F.SilkS) (width 0.12))
+    (fp_line (start -1.96 -0.7) (end 1.95 -0.7) (layer F.CrtYd) (width 0.05))
+    (fp_line (start -1.96 -0.7) (end -1.96 0.7) (layer F.CrtYd) (width 0.05))
+    (fp_line (start 1.95 0.7) (end 1.95 -0.7) (layer F.CrtYd) (width 0.05))
+    (fp_line (start 1.95 0.7) (end -1.96 0.7) (layer F.CrtYd) (width 0.05))
+    (pad 1 smd rect (at -1.1 0 180) (size 1.2 0.9) (layers F.Cu F.Paste F.Mask)
+      (net 3 "Net-(J1-Pad1)"))
+    (pad 2 smd rect (at 1.1 0 180) (size 1.2 0.9) (layers F.Cu F.Paste F.Mask)
+      (net 2 "Net-(D1-Pad2)"))
+    (model ${KISYS3DMOD}/Resistors_SMD.3dshapes/R_0603.wrl
+      (at (xyz 0 0 0))
+      (scale (xyz 1 1 1))
+      (rotate (xyz 0 0 0))
+    )
+  )
+  (module LEDs:LED_0603_HandSoldering (layer F.Cu)
+    (at 118.745 90.17 180)
+    (descr "LED SMD 0603, hand soldering")
+    (tags "LED 0603")
+    (attr smd)
+    (fp_text reference D1 (at 0 -1.45 180) (layer F.SilkS)
+      (effects (font (size 1 1) (thickness 0.15)))
+    )
+    (fp_text value LED (at 0 1.55 180) (layer F.Fab)
+      (effects (font (size 1 1) (thickness 0.15)))
+    )
+    (fp_line (start -1.8 -0.55) (end -1.8 0.55) (layer F.SilkS) (width 0.12))
+    (fp_line (start -0.2 -0.2) (end -0.2 0.2) (layer F.Fab) (width 0.1))
+    (fp_line (start -0.15 0) (end 0.15 -0.2) (layer F.Fab) (width 0.1))
+    (fp_line (start 0.15 0.2) (end -0.15 0) (layer F.Fab) (width 0.1))
+    (fp_line (start 0.15 -0.2) (end 0.15 0.2) (layer F.Fab) (width 0.1))
+    (fp_line (start 0.8 0.4) (end -0.8 0.4) (layer F.Fab) (width 0.1))
+    (fp_line (start 0.8 -0.4) (end 0.8 0.4) (layer F.Fab) (width 0.1))
+    (fp_line (start -0.8 -0.4) (end 0.8 -0.4) (layer F.Fab) (width 0.1))
+    (fp_line (start -1.8 0.55) (end 0.8 0.55) (layer F.SilkS) (width 0.12))
+    (fp_line (start -1.8 -0.55) (end 0.8 -0.55) (layer F.SilkS) (width 0.12))
+    (fp_line (start -1.96 -0.7) (end 1.95 -0.7) (layer F.CrtYd) (width 0.05))
+    (fp_line (start -1.96 -0.7) (end -1.96 0.7) (layer F.CrtYd) (width 0.05))
+    (fp_line (start 1.95 0.7) (end 1.95 -0.7) (layer F.CrtYd) (width 0.05))
+    (fp_line (start 1.95 0.7) (end -1.96 0.7) (layer F.CrtYd) (width 0.05))
+    (fp_line (start -0.8 -0.4) (end -0.8 0.4) (layer F.Fab) (width 0.1))
+    (pad 1 smd rect (at -1.1 0 180) (size 1.2 0.9) (layers F.Cu F.Paste F.Mask)
+      (net 1 GND))
+    (pad 2 smd rect (at 1.1 0 180) (size 1.2 0.9) (layers F.Cu F.Paste F.Mask)
+      (net 2 "Net-(D1-Pad2)"))
+    (model ${KISYS3DMOD}/LEDs.3dshapes/LED_0603.wrl
+      (at (xyz 0 0 0))
+      (scale (xyz 1 1 1))
+      (rotate (xyz 0 0 180))
+    )
+  )
   (gr_line (start 133.04972 78.282406) (end 132.584777 78.285267) (layer Edge.Cuts) (width 0.1))
   (gr_line (start 132.584777 78.285267) (end 132.121327 78.302593) (layer Edge.Cuts) (width 0.1))
@@
   (gr_line (start 133.04972 78.282406) (end 133.04972 78.282406) (layer Edge.Cuts) (width 0.1))
   (gr_line (start 133.04972 78.282406) (end 133.04972 78.282406) (layer Edge.Cuts) (width 0.1))
+  (segment (start 119.845 90.17) (end 120.015 90.17) (width 0.25) (layer F.Cu) (net 1) (status C00000))
+  (segment (start 120.015 90.17) (end 122.555 92.71) (width 0.25) (layer F.Cu) (net 1) (status 400000))
+  (segment (start 122.555 92.71) (end 127.635 92.71) (width 0.25) (layer F.Cu) (net 1))
+  (segment (start 127.635 92.71) (end 131.39 88.955) (width 0.25) (layer F.Cu) (net 1))
+  (segment (start 131.39 88.955) (end 131.39 86.53) (width 0.25) (layer F.Cu) (net 1) (status 800000))
+  (segment (start 111.93 86.36) (end 111.93 87.46) (width 0.25) (layer F.Cu) (net 2) (status 400000))
+  (segment (start 116.375 88.9) (end 117.645 90.17) (width 0.25) (layer F.Cu) (net 2) (status 800000))
+  (segment (start 113.37 88.9) (end 116.375 88.9) (width 0.25) (layer F.Cu) (net 2))
+  (segment (start 111.93 87.46) (end 113.37 88.9) (width 0.25) (layer F.Cu) (net 2))
+  (segment (start 114.13 86.36) (end 117.475 86.36) (width 0.25) (layer F.Cu) (net 3) (status 400000))
+  (segment (start 129.37 83.99) (end 131.39 83.99) (width 0.25) (layer F.Cu) (net 3) (status 800000))
+  (segment (start 128.27 85.09) (end 129.37 83.99) (width 0.25) (layer F.Cu) (net 3))
+  (segment (start 128.27 86.36) (end 128.27 85.09) (width 0.25) (layer F.Cu) (net 3))
+  (segment (start 128.27 90.805) (end 128.27 86.36) (width 0.25) (layer F.Cu) (net 3))
+  (segment (start 127 92.075) (end 128.27 90.805) (width 0.25) (layer F.Cu) (net 3))
+  (segment (start 123.19 92.075) (end 127 92.075) (width 0.25) (layer F.Cu) (net 3))
+  (segment (start 122.555 91.44) (end 123.19 92.075) (width 0.25) (layer F.Cu) (net 3))
+  (segment (start 122.555 90.805) (end 122.555 91.44) (width 0.25) (layer F.Cu) (net 3))
+  (segment (start 121.92 90.17) (end 122.555 90.805) (width 0.25) (layer F.Cu) (net 3))
+  (segment (start 121.92 89.535) (end 121.92 90.17) (width 0.25) (layer F.Cu) (net 3))
+  (segment (start 121.285 88.9) (end 121.92 89.535) (width 0.25) (layer F.Cu) (net 3))
+  (segment (start 119.38 86.995) (end 121.285 88.9) (width 0.25) (layer F.Cu) (net 3))
+  (segment (start 118.745 86.995) (end 119.38 86.995) (width 0.25) (layer F.Cu) (net 3))
+  (segment (start 118.11 86.36) (end 118.745 86.995) (width 0.25) (layer F.Cu) (net 3))
+  (segment (start 117.475 86.36) (end 118.11 86.36) (width 0.25) (layer F.Cu) (net 3))
 )

Commit message: tweaking on the led
Parts:
- removed the ? at (153.1, 107.2)
- added ?: , un1eet_sao:F.Mask_g8167, B.Cu at (153.5, 82.3)
- D1, R1: moved to B.Cu
- moved R1 13.7 mm to (125.4, 92.4)
- moved D1 8.88 mm to (111.0, 94.5)
- moved ? 2.62 mm to (153.2, 109.8)
- moved ? 0.75 mm to (153.5, 106.6)
Routing:
- net GND: track 16.6 -> 33.4 mm
- net Net-(J1-Pad1): track 27.1 -> 10.5 mm
- net Net-(D1-Pad2): track 7.94 -> 15.3 mm

Commit message: cleaned up design
Routing:
- added copper zone on F.Cu, net GND
Changed lines of the file:
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@@
     (links 3)
     (no_connects 0)
-    (area 103.86345 78.232405 202.022987 111.2742)
+    (area 92.645147 67.705995 209.160001 114.440001)
     (thickness 1.6)
     (drawings 1059)
@@
     (trace_clearance 0.2)
     (zone_clearance 0.508)
-    (zone_45_only no)
+    (zone_45_only yes)
     (trace_min 0.2)
     (segment_width 0.2)
@@
   (segment (start 129.14 86.08) (end 129.14 89.72) (width 0.25) (layer B.Cu) (net 3))
   (segment (start 129.14 89.72) (end 126.49 92.37) (width 0.25) (layer B.Cu) (net 3))
+  (zone (net 1) (net_name GND) (layer F.Cu) (hatch edge 0.508)
+    (connect_pads (clearance 0.508))
+    (min_thickness 0.254)
+    (fill yes (arc_segments 16) (thermal_gap 0.508) (thermal_bridge_width 0.508))
+    (polygon
+      (pts
+        (xy 100.53 92.03) (xy 112.65 75.38) (xy 209.16 86.45) (xy 201.39 114.44) (xy 103.83 113.83)
+      )
+    )
+  )
+  (zone (net 0) (net_name "") (layer F.Cu) (hatch edge 0.508)
+    (connect_pads (clearance 0.508))
+    (min_thickness 0.254)
+    (keepout (tracks not_allowed) (vias not_allowed) (copperpour allowed))
+    (fill (arc_segments 16) (thermal_gap 0.508) (thermal_bridge_width 0.508))
+    (polygon
+      (pts
+        (xy 141.77 89.6) (xy 140.04 89.6) (xy 139.42 90.22) (xy 128.86 90.22) (xy 128.36 90.72)
+        (xy 126.37 90.72) (xy 124.14 88.49) (xy 124.14 76.44) (xy 142.21 76.44) (xy 142.21 77.39)
+      )
+    )
+  )
 )
